File: sd-card.kicad_sch (KiCad schematic)
At the start: 6 parts, among them J1 Micro_SD_Card_Det_Hirose_DM3AT

Commit message: Finished SDRAM, QSPI Flash, Planning to move to 5 inch orient display dimension
Parts:
- J1: JLCPCB Part # C114218 -> C597972
Changed lines of the file:
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@@
 			)
 		)
-		(property "JLCPCB Part #" "C114218"
+		(property "JLCPCB Part #" "C597972"
 			(at 165.1 97.79 0)
 			(effects
