File: sd-card.kicad_sch (KiCad schematic)
At the start: 6 parts, among them J6 Micro_SD_Card_Det1

Commit message: Almost finished
Parts:
- J6: JLCPCB Part # (none) -> C266621
Changed lines of the file:
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@@
+			)
+		)
+		(property "JLCPCB Part #" "C266621"
+			(at 157.48 96.52 0)
+			(effects
+				(font
+					(size 1.27 1.27)
+				)
+				(hide yes)
 			)
 		)
