File: MAX98357.kicad_sch (KiCad schematic)
At the start: 20 parts, among them J11 AudioJack3, J8 SPKR, U10 PCM5102A, U6 MAX98357AETE_

Commit message: Almost finished
Parts:
- R15: now not fitted; now left out of the parts list
- R16: value NC -> 100K; JLCPCB Part # (none) -> C60491
Changed lines of the file:
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@@
 			)
 		)
-		(property "Value" "NC"
+		(property "Value" "100K"
 			(at 64.77 146.0499 0)
 			(effects
@@
 			)
 		)
-		(property "JLCPCB Part #" ""
+		(property "JLCPCB Part #" "C60491"
 			(at 62.23 144.78 0)
 			(effects
@@
 		(unit 1)
 		(exclude_from_sim no)
-		(in_bom yes)
-		(on_board yes)
-		(dnp no)
+		(in_bom no)
+		(on_board yes)
+		(dnp yes)
 		(fields_autoplaced yes)
 		(property "Reference" "R15"
