File: MAX98357.kicad_sch (KiCad schematic)
At the start: 20 parts, among them J11 AudioJack3, J8 SPKR, U10 PCM5102A, U6 MAX98357AETE_

Commit message: Still on progress...
Parts:
- added C68: 100n, Capacitor_SMD:C_0402_1005Metric, symbol Device:C_Small
- J11: footprint Connector_Audio:Jack_3.5mm_CUI_SJ-3523-SMT_Horizontal -> Audio-jack-3_5mm-custom:XKB-PJ-320B-SMT
Connections:
- net +3V3: now also U10.17 (XSMT)
- net GND: now also U10.10 (DEMP), U10.11 (FLT), U10.12 (SCK), U10.16 (FMT), C68.2
- net at U10.18 (LDOO): now also C68.1
- net BCK renamed I2S2_CK
- net DIN renamed I2S2_DIN
- net I2S_CK renamed I2S3_CK
- net I2S_SDO renamed I2S3_SDO
- net I2S_SD_MODE renamed I2S3_SD_MODE
- net I2S_WS renamed I2S3_WS
- net LRCK renamed I2S2_WS
