File: nor-flash.kicad_sch (KiCad schematic)
At the start: 6 parts, among them U1 MT25Q, U4 MT25Q

Commit message: not yet
Parts:
- added JP8: FLASH_CONFIG, Jumper:SolderJumper-3_P1.3mm_Open_RoundedPad1.0x1.5mm_NumberLabels, symbol Jumper:SolderJumper_3_Open
- added JP9: FLASH_EN, Jumper:SolderJumper-2_P1.3mm_Open_RoundedPad1.0x1.5mm, symbol Jumper:SolderJumper_2_Open
Connections:
- net +3V3: now also JP9.2 (B); no longer C22.1, U4.8 (VCC)
- net QUADSPI_BK1_NCS: now also JP8.3 (B)
- net QUADSPI_BK2_NCS: now also JP8.1 (A); no longer R2.2, U4.1 (~{CS})
- new net: C22.1, JP9.1 (A), U4.8 (VCC)
- new net: JP8.2 (C), R2.2, U4.1 (~{CS})
