File: chroma-pixel-zeta.kicad_sch (KiCad schematic)
At the start: 4 parts

Commit message: Almost finished
Other:
- sheet LCD ports: added LCD_SPI_CS; removed none
- sheet MCU ports: added LCD_SPI_CS; removed none
Changed lines of the file:
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@@
 	(wire
 		(pts
-			(xy 58.42 72.39) (xy 74.93 72.39)
+			(xy 58.42 76.2) (xy 74.93 76.2)
 		)
 		(stroke
@@
 	(wire
 		(pts
-			(xy 58.42 67.31) (xy 74.93 67.31)
+			(xy 58.42 68.58) (xy 74.93 68.58)
 		)
 		(stroke
@@
 	(wire
 		(pts
-			(xy 58.42 69.85) (xy 74.93 69.85)
+			(xy 58.42 73.66) (xy 74.93 73.66)
 		)
 		(stroke
@@
 		)
 	)
+	(wire
+		(pts
+			(xy 58.42 71.12) (xy 74.93 71.12)
+		)
+		(stroke
+			(width 0)
+			(type default)
+		)
+	)
 	(bus
 		(pts
@@
 	(wire
 		(pts
-			(xy 58.42 74.93) (xy 74.93 74.93)
+			(xy 58.42 78.74) (xy 74.93 78.74)
 		)
 		(stroke
@@
 	(wire
 		(pts
-			(xy 58.42 85.09) (xy 74.93 85.09)
+			(xy 58.42 88.9) (xy 74.93 88.9)
 		)
 		(stroke
@@
 	(wire
 		(pts
-			(xy 58.42 82.55) (xy 74.93 82.55)
+			(xy 58.42 86.36) (xy 74.93 86.36)
 		)
 		(stroke
@@
 	(wire
 		(pts
-			(xy 58.42 80.01) (xy 74.93 80.01)
+			(xy 58.42 83.82) (xy 74.93 83.82)
 		)
 		(stroke
@@
 		)
 		(pin "LCD_SPI_MISO" input
-			(at 74.93 74.93 180)
+			(at 74.93 78.74 180)
 			(effects
 				(font
@@
 		)
 		(pin "LCD_SPI_SCK" output
-			(at 74.93 69.85 180)
+			(at 74.93 73.66 180)
 			(effects
 				(font
@@
 		)
 		(pin "LCD_SPI_MOSI" output
-			(at 74.93 72.39 180)
+			(at 74.93 76.2 180)
 			(effects
 				(font
@@
 		)
 		(pin "LCD_SPI_DC" output
-			(at 74.93 67.31 180)
+			(at 74.93 68.58 180)
 			(effects
 				(font
@@
 		)
 		(pin "LCD_SPI_CLK" output
-			(at 74.93 80.01 180)
+			(at 74.93 83.82 180)
 			(effects
 				(font
@@
 		)
 		(pin "LCD_SPI_DAT" bidirectional
-			(at 74.93 82.55 180)
+			(at 74.93 86.36 180)
 			(effects
 				(font
@@
 		)
 		(pin "LCD_SPI_RESET" output
-			(at 74.93 85.09 180)
+			(at 74.93 88.9 180)
+			(effects
+				(font
+					(size 1.27 1.27)
+				)
+				(justify left)
+			)
+		)
+		(pin "LCD_SPI_CS" output
+			(at 74.93 71.12 180)
 			(effects
 				(font
@@
 		)
 		(pin "LCD_SPI_MISO" output
-			(at 58.42 74.93 0)
+			(at 58.42 78.74 0)
 			(effects
 				(font
@@
 		)
 		(pin "LCD_SPI_DC" input
-			(at 58.42 67.31 0)
+			(at 58.42 68.58 0)
 			(effects
 				(font
@@
 		)
 		(pin "LCD_SPI_MOSI" input
-			(at 58.42 72.39 0)
+			(at 58.42 76.2 0)
 			(effects
 				(font
@@
 		)
 		(pin "LCD_SPI_SCK" input
-			(at 58.42 69.85 0)
+			(at 58.42 73.66 0)
 			(effects
 				(font
@@
 		)
 		(pin "LCD_SPI_CLK" input
-			(at 58.42 80.01 0)
+			(at 58.42 83.82 0)
 			(effects
 				(font
@@
 		)
 		(pin "LCD_SPI_DAT" bidirectional
-			(at 58.42 82.55 0)
+			(at 58.42 86.36 0)
 			(effects
 				(font
@@
 		)
 		(pin "LCD_SPI_RESET" input
-			(at 58.42 85.09 0)
-			(effects
-				(font
+			(at 58.42 88.9 0)
+			(effects
+				(font
+					(size 1.27 1.27)
+				)
+				(justify right)
+			)
+		)
+		(pin "LCD_SPI_CS" input
+			(at 58.42 71.12 0)
+			(effects
+				(font

Commit message: Still on progress...
Other:
- sheet AUDIO ports: added I2S2_CK, I2S2_DIN, I2S2_WS, I2S3_CK, I2S3_SDO, I2S3_SD_MODE, I2S3_WS; removed I2S_CK, I2S_SDO, I2S_SD_MODE, I2S_WS
- sheet DCMI ports: added CAM_SCL, CAM_SDA; removed none
- sheet MCU ports: added I2S2_CK, I2S2_DIN, I2S2_WS, I2S3_CK, I2S3_SDO, I2S3_SD_MODE, I2S3_WS; removed I2S_CK, I2S_SDO, I2S_SD_MODE, I2S_WS
