File: chroma-pixel-zeta.kicad_sch (KiCad schematic)
At the start: 4 parts

Commit message: First release
Other:
- sheet DCMI ports: added none; removed CAM_SCL, CAM_SDA, DCMI_D[0..7], DCMI_HSYNC, DCMI_PIXCLK, DCMI_VSYNC
- sheet MCU ports: added VBUS_EN; removed DCMI_D[0..7], DCMI_HSYNC, DCMI_PIXCLK, DCMI_VSYNC
- sheet USB ports: added USB_OVCR, USB_PWR_EN, VBUS_SENS; removed none
